Commit message: Lidar pos

File: urdf/rosgolf_robot.urdf (robot description, URDF)
Before this commit: robot rosgolf_robot, 9 links, 8 joints
Joints:
- joint base_to_scanner: origin xyz=0.0 -0.04 0.26 rpy=0 0 0 -> xyz=0.0 -0.04 0.26 rpy=0 3.14 0

Commit message: Lidar pos

File: urdf/rosgolf_robot.urdf (robot description, URDF)
Before this commit: robot rosgolf_robot, 9 links, 8 joints
Joints:
- joint base_to_scanner: origin xyz=0.0 -0.04 0.26 rpy=0 3.14 0 -> xyz=0.0 0.0 0.26 rpy=0 0 3.14
